File: eagle/kriner-pc.brd (EAGLE design)
At the start: 38.1 x 38.1 mm, 16 parts, among them Q1 FJN3305RTA, Q2 FQP27P06

Commit message: Closes #1.
Other:
- board text added: "1.1"
Changed lines of the file:
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@@
 <text x="34.925" y="35.56" size="1.27" layer="22" rot="MR0">github.com/gregkrsak/kriner-pc</text>
 <text x="27.4066" y="17.1196" size="1.27" layer="22" rot="MR0">CC BY-SA 3.0 US</text>
+<text x="2.794" y="0.254" size="1.27" layer="22" rot="MR0">1.1</text>
 </plain>
 <attributes>
@@
 </signal>
 <signal name="V+">
-<contactref element="R1" pad="P$2"/>
-<contactref element="Q2" pad="3"/>
-<contactref element="JP2-1" pad="1"/>
-<contactref element="S2" pad="4"/>
-<contactref element="S1" pad="2"/>
 <contactref element="JP1" pad="1"/>
-<wire x1="21.59" y1="9.8425" x2="35.2425" y2="9.8425" width="2.54" layer="16"/>
-<wire x1="21.59" y1="9.9219" x2="21.59" y2="9.8425" width="2.54" layer="16"/>
-<wire x1="21.59" y1="9.9219" x2="21.59" y2="11.0331" width="2.54" layer="16"/>
-<wire x1="15.9512" y1="7.0231" x2="18.6912" y2="7.0231" width="0.3048" layer="16"/>
-<wire x1="18.6912" y1="7.0231" x2="21.59" y2="9.9219" width="0.3048" layer="16"/>
-<wire x1="35.2425" y1="9.0932" x2="28.6512" y2="2.5019" width="0.3048" layer="16"/>
-<wire x1="35.2425" y1="9.8425" x2="35.2425" y2="9.0932" width="0.3048" layer="16"/>
-<wire x1="10.5569" y1="12.4174" x2="15.9512" y2="7.0231" width="0.3048" layer="16"/>
-<wire x1="10.5569" y1="12.5413" x2="10.5569" y2="12.4174" width="0.3048" layer="16"/>
-<wire x1="4.2069" y1="18.8913" x2="10.5569" y2="12.5413" width="0.3048" layer="1"/>
-<wire x1="1.5081" y1="18.8913" x2="4.2069" y2="18.8913" width="0.3048" layer="1"/>
-<wire x1="0.635" y1="19.7644" x2="1.5081" y2="18.8913" width="0.3048" layer="1"/>
-<wire x1="0.635" y1="19.7644" x2="0.635" y2="28.7654" width="0.3048" layer="1"/>
-<wire x1="0.635" y1="28.7654" x2="2.3495" y2="30.4799" width="0.3048" layer="1"/>
 <polygon width="0.3048" layer="16" isolate="0.3048" thermals="no">
 <vertex x="0" y="0"/>
@@
 <vertex x="0" y="12.7"/>
 </polygon>
+<contactref element="R1" pad="P$2"/>
+<contactref element="S2" pad="4"/>
+<contactref element="S1" pad="2"/>
+<wire x1="10.5569" y1="12.4174" x2="15.9512" y2="7.0231" width="0.3048" layer="16"/>
+<wire x1="10.5569" y1="12.5413" x2="10.5569" y2="12.4174" width="0.3048" layer="16"/>
+<contactref element="Q2" pad="3"/>
+<wire x1="15.9512" y1="7.0231" x2="19.7231" y2="7.0231" width="0.3048" layer="16"/>
+<wire x1="19.7231" y1="7.0231" x2="21.59" y2="8.89" width="0.3048" layer="16"/>
+<wire x1="21.59" y1="8.89" x2="21.59" y2="11.0331" width="0.3048" layer="16"/>
+<wire x1="21.59" y1="11.0331" x2="23.7649" y2="11.0331" width="0.3048" layer="16"/>
+<wire x1="23.7649" y1="11.0331" x2="25.654" y2="9.144" width="0.3048" layer="16"/>
+<wire x1="25.654" y1="9.144" x2="25.654" y2="5.4991" width="0.3048" layer="16"/>
+<wire x1="25.654" y1="5.4991" x2="28.6512" y2="2.5019" width="0.3048" layer="16"/>
+<wire x1="2.3495" y1="30.4799" x2="1.5239" y2="30.4799" width="0.3048" layer="1"/>
+<wire x1="1.5239" y1="30.4799" x2="0.762" y2="29.718" width="0.3048" layer="1"/>
+<wire x1="0.762" y1="29.718" x2="0.762" y2="19.812" width="0.3048" layer="1"/>
+<wire x1="0.762" y1="19.812" x2="2.286" y2="18.288" width="0.3048" layer="1"/>
+<wire x1="2.286" y1="18.288" x2="4.8102" y2="18.288" width="0.3048" layer="1"/>
+<wire x1="4.8102" y1="18.288" x2="10.5569" y2="12.5413" width="0.3048" layer="1"/>
+<contactref element="JP2-1" pad="1"/>
+<wire x1="25.654" y1="9.144" x2="34.544" y2="9.144" width="0.3048" layer="16"/>
+<wire x1="34.544" y1="9.144" x2="35.2425" y2="9.8425" width="0.3048" layer="16"/>
 </signal>
 <signal name="V-">
@@
 <wire x1="5.9531" y1="12.5412" x2="8.2551" y2="12.5412" width="0.3048" layer="16"/>
 <wire x1="16.51" y1="10.0013" x2="16.51" y2="10.0806" width="0.3048" layer="1"/>
-<wire x1="16.51" y1="10.4775" x2="16.51" y2="11.0331" width="0.3048" layer="1"/>
+<wire x1="16.51" y1="10.0806" x2="16.51" y2="11.0331" width="0.3048" layer="1"/>
 <wire x1="11.3506" y1="4.8419" x2="16.51" y2="10.0013" width="0.3048" layer="1"/>
 <wire x1="7.2231" y1="4.8419" x2="11.3506" y2="4.8419" width="0.3048" layer="1"/>
@@
 <wire x1="21.1931" y1="5.3975" x2="23.0981" y2="5.3975" width="0.3048" layer="1"/>
 <wire x1="16.51" y1="10.0806" x2="21.1931" y2="5.3975" width="0.3048" layer="1"/>
-<wire x1="16.51" y1="10.0806" x2="16.51" y2="10.4775" width="0.3048" layer="1"/>
 </signal>
 </signals>
